Commit message: update human model

File: tests/files/human165.urdf (robot description, URDF)
Before this commit: robot human, 27 links, 26 joints
Links:
- removed link body_default
- removed link l_ankle_default
- removed link l_elbow_default
- removed link l_hip_default
- removed link l_knee_default
- removed link l_p_hip_default
- removed link l_p_shoulder_default
- removed link l_shoulder_default
- removed link l_wrist_default
- removed link l_y_hip_default
- removed link l_y_shoulder_default
- removed link r_ankle_default
- removed link r_elbow_default
- removed link r_hip_default
- removed link r_knee_default
- removed link r_p_hip_default
- removed link r_p_shoulder_default
- removed link r_shoulder_default
- removed link r_wrist_default
- removed link r_y_hip_default
- removed link r_y_shoulder_default
- removed link torso_default
- added link body_root_default
- added link chest_default; visual cylinder length=0.1872340425531915 radius=0.03; visual cylinder length=0.1872340425531915 radius=0.03
- added link left_foot_default
- added link left_forearm_default; visual cylinder length=0.22 radius=0.03; visual sphere radius=0.03
- added link left_hand_default
- added link left_p_hip_default
- added link left_p_shoulder_default
- added link left_shank_default; visual cylinder length=0.44 radius=0.03; visual sphere radius=0.03
- added link left_thigh_default; visual cylinder length=0.33 radius=0.03; visual sphere radius=0.03
- added link left_upper_arm_default; visual cylinder length=0.35200000000000004 radius=0.03; visual sphere radius=0.03
- added link left_y_hip_default; visual sphere radius=0.03
- added link left_y_shoulder_default; visual sphere radius=0.03
- added link right_foot_default
- added link right_forearm_default; visual cylinder length=0.22 radius=0.03; visual sphere radius=0.03
- added link right_hand_default
- added link right_p_hip_default
- added link right_p_shoulder_default
- added link right_shank_default; visual cylinder length=0.44 radius=0.03; visual sphere radius=0.03
- added link right_thigh_default; visual cylinder length=0.33 radius=0.03; visual sphere radius=0.03
- added link right_upper_arm_default; visual cylinder length=0.35200000000000004 radius=0.03; visual sphere radius=0.03
- added link right_y_hip_default; visual sphere radius=0.03
- added link right_y_shoulder_default; visual sphere radius=0.03
Joints:
- removed joint head_default
- removed joint l_ankle_default
- removed joint l_elbow_default
- removed joint l_knee_default
- removed joint l_p_hip_default
- removed joint l_p_shoulder_default
- removed joint l_r_hip_default
- removed joint l_r_shoulder_default
- removed joint l_wrist_default
- removed joint l_y_hip_default
- removed joint l_y_shoulder_default
- removed joint p_head_default
- removed joint r_ankle_default
- removed joint r_elbow_default
- removed joint r_head_default
- removed joint r_knee_default
- removed joint r_p_hip_default
- removed joint r_p_shoulder_default
- removed joint r_r_hip_default
- removed joint r_r_shoulder_default
- removed joint r_wrist_default
- removed joint r_y_hip_default
- removed joint r_y_shoulder_default
- removed joint torso_default
- removed joint waist_default
- removed joint y_head_default
- added joint head_fixed_default: type fixed, parent p_head_default, child head_default, origin xyz=0.055 0 0.11 rpy=0 0 0
- added joint left_ankle_default: type fixed, parent left_shank_default, child left_foot_default, origin xyz=0 0 -0.44 rpy=0 0 0
- added joint left_elbow_flx_default: type revolute, parent left_upper_arm_default, child left_forearm_default, origin xyz=0 0 -0.35200000000000004 rpy=0 0 0, axis 0 -1 0, limit lower=0 upper=2.5 effort=1000 velocity=0.5
- added joint left_flx_shoulder_default: type revolute, parent left_y_shoulder_default, child left_p_shoulder_default, origin xyz=0 0 0 rpy=0 0 0, axis 1 0 0, limit lower=-0.4 upper=3.3 effort=1000 velocity=0.5
- added joint left_hip=rot_default: type revolute, parent left_p_hip_default, child left_thigh_default, origin xyz=0 0 0 rpy=0 0 0, axis 0 -1 0, limit lower=-0.7 upper=0.7 effort=1000 velocity=0.5
- added joint left_hip_add_default: type revolute, parent body_root_default, child left_y_hip_default, origin xyz=0 0.132 0 rpy=0 0 0, axis 0 0  -1.0, limit lower=-0.87 upper=0.5 effort=1000 velocity=0.5
- added joint left_hip_flx_default: type revolute, parent left_y_hip_default, child left_p_hip_default, origin xyz=0 0 0 rpy=0 0 0, axis 1 0 0, limit lower=-0.5 upper=2.1 effort=1000 velocity=0.5
- added joint left_knee_flx_default: type revolute, parent left_thigh_default, child left_shank_default, origin xyz=0 0 -0.33 rpy=0 0 0, axis 0 1 0, limit lower=0 upper=2.5 effort=1000 velocity=0.5
- added joint left_shoulder_add_default: type revolute, parent chest_default, child left_y_shoulder_default, origin xyz=0 0.17600000000000002 0 rpy=0 0 0, axis 0 0 -1, limit lower=-1.7 upper=1.1 effort=1000 velocity=0.5
- added joint left_shoulder_rot_default: type revolute, parent left_p_shoulder_default, child left_upper_arm_default, origin xyz=0 0 0 rpy=0 0 0, axis 0 0 1, limit lower=-1.7 upper=1.5 effort=1000 velocity=0.5
- added joint left_wrist_fixed_default: type fixed, parent left_forearm_default, child left_hand_default, origin xyz=0 0 -0.22 rpy=0 0 0
- added joint lumbar_default: type fixed, parent waist_default, child chest_default, origin xyz=0 0 0.605 rpy=0 0 0
- added joint pitch_head_default: type revolute, parent y_head_default, child p_head_default, origin xyz=0 0 0 rpy=0 0 0, axis 0 -1 0, limit lower=-1.5 upper=1.5 effort=1000 velocity=0.5
- added joint right_ankle_default: type fixed, parent right_shank_default, child right_foot_default, origin xyz=0 0 -0.44 rpy=0 0 0
- added joint right_elbow_flx_default: type revolute, parent right_upper_arm_default, child right_forearm_default, origin xyz=0 0 -0.35200000000000004 rpy=0 0 0, axis 0 -1 0, limit lower=0 upper=2.5 effort=1000 velocity=0.5
- added joint right_flx_shoulder_default: type revolute, parent right_y_shoulder_default, child right_p_shoulder_default, origin xyz=0 0 0 rpy=0 0 0, axis -1 0 0, limit lower=-0.4 upper=3.3 effort=1000 velocity=0.5
- added joint right_hip=rot_default: type revolute, parent right_p_hip_default, child right_thigh_default, origin xyz=0 0 0 rpy=0 0 0, axis 0 -1 0, limit lower=-0.7 upper=0.7 effort=1000 velocity=0.5
- added joint right_hip_add_default: type revolute, parent body_root_default, child right_y_hip_default, origin xyz=0 -0.132 0 rpy=0 0 0, axis 0 0  1.0, limit lower=-0.87 upper=0.5 effort=1000 velocity=0.5
- added joint right_hip_flx_default: type revolute, parent right_y_hip_default, child right_p_hip_default, origin xyz=0 0 0 rpy=0 0 0, axis -1 0 0, limit lower=-0.5 upper=2.1 effort=1000 velocity=0.5
- added joint right_knee_flx_default: type revolute, parent right_thigh_default, child right_shank_default, origin xyz=0 0 -0.33 rpy=0 0 0, axis 0 1 0, limit lower=0 upper=2.5 effort=1000 velocity=0.5
- added joint right_shoulder_add_default: type revolute, parent chest_default, child right_y_shoulder_default, origin xyz=0 -0.17600000000000002 0 rpy=0 0 0, axis 0 0 1, limit lower=-1.7 upper=1.1 effort=1000 velocity=0.5
- added joint right_shoulder_rot_default: type revolute, parent right_p_shoulder_default, child right_upper_arm_default, origin xyz=0 0 0 rpy=0 0 0, axis 0 0 -1, limit lower=-1.7 upper=1.5 effort=1000 velocity=0.5
- added joint right_wrist_fixed_default: type fixed, parent right_forearm_default, child right_hand_default, origin xyz=0 0 -0.22 rpy=0 0 0
- added joint roll_head_default: type revolute, parent chest_default, child r_head_default, origin xyz=0 0 0.055 rpy=0 0 0, axis 1 0 0, limit lower=-1. upper=1. effort=1000 velocity=0.5
- added joint spine_default: type revolute, parent body_root_default, child waist_default, origin xyz=0 0 0 rpy=0 0 0, axis 0 1 0, limit lower=-.2 upper=1. effort=1000 velocity=0.5
- added joint yaw_head_default: type revolute, parent r_head_default, child y_head_default, origin xyz=0 0 0 rpy=0 0 0, axis 0 0 1, limit lower=-1.4 upper=1.4 effort=1000 velocity=0.5

Commit message: update human model

File: tests/files/human165.urdf (robot description, URDF)
Before this commit: robot human, 27 links, 26 joints
Joints:
- removed joint left_flx_shoulder_default
- removed joint left_hip=rot_default
- removed joint left_shoulder_add_default
- removed joint right_flx_shoulder_default
- removed joint right_hip=rot_default
- removed joint right_shoulder_add_default
- added joint left_add_shoulder_default: type revolute, parent left_y_shoulder_default, child left_p_shoulder_default, origin xyz=0 0 0 rpy=0 0 0, axis -1 0 0, limit lower=-1.7 upper=1.1 effort=1000 velocity=0.5
- added joint left_hip_rot_default: type revolute, parent left_p_hip_default, child left_thigh_default, origin xyz=0 0 0 rpy=0 0 0, axis 0 0 -1, limit lower=-0.7 upper=0.7 effort=1000 velocity=0.5
- added joint left_shoulder_flx_default: type revolute, parent chest_default, child left_y_shoulder_default, origin xyz=0 0.17600000000000002 0 rpy=0 0 0, axis 0 -1 0, limit lower=-0.4 upper=3.3 effort=1000 velocity=0.5
- added joint right_add_shoulder_default: type revolute, parent right_y_shoulder_default, child right_p_shoulder_default, origin xyz=0 0 0 rpy=0 0 0, axis 1 0 0, limit lower=-1.7 upper=1.1 effort=1000 velocity=0.5
- added joint right_hip_rot_default: type revolute, parent right_p_hip_default, child right_thigh_default, origin xyz=0 0 0 rpy=0 0 0, axis 0 0 1, limit lower=-0.7 upper=0.7 effort=1000 velocity=0.5
- added joint right_shoulder_flx_default: type revolute, parent chest_default, child right_y_shoulder_default, origin xyz=0 -0.17600000000000002 0 rpy=0 0 0, axis 0 -1 0, limit lower=-0.4 upper=3.3 effort=1000 velocity=0.5
- joint left_hip_add_default: axis 0 0  -1.0 -> -1 0 0; child left_y_hip_default -> left_p_hip_default; origin xyz=0 0.132 0 rpy=0 0 0 -> xyz=0 0 0 rpy=0 0 0; parent body_root_default -> left_y_hip_default
- joint left_hip_flx_default: axis 1 0 0 -> 0 -1 0; child left_p_hip_default -> left_y_hip_default; origin xyz=0 0 0 rpy=0 0 0 -> xyz=0 0.132 0 rpy=0 0 0; parent left_y_hip_default -> body_root_default
- joint left_shoulder_rot_default: axis 0 0 1 -> 0 0 -1
- joint right_hip_add_default: axis 0 0  1.0 -> 1 0 0; child right_y_hip_default -> right_p_hip_default; origin xyz=0 -0.132 0 rpy=0 0 0 -> xyz=0 0 0 rpy=0 0 0; parent body_root_default -> right_y_hip_default
- joint right_hip_flx_default: axis -1 0 0 -> 0 -1 0; child right_p_hip_default -> right_y_hip_default; origin xyz=0 0 0 rpy=0 0 0 -> xyz=0 -0.132 0 rpy=0 0 0; parent right_y_hip_default -> body_root_default
- joint right_shoulder_rot_default: axis 0 0 -1 -> 0 0 1
