Commit message: update ik

File: tests/files/human-xyz-165.urdf (robot description, URDF)
Before this commit: robot human, 34 links, 33 joints
Joints:
- joint rail_x_default: limit lower=-2.5 upper=2.5 effort=1000 velocity=0.5 -> lower=-10 upper=10 effort=1000 velocity=0.5
- joint rail_y_default: limit lower=-2.5 upper=2.5 effort=1000 velocity=0.5 -> lower=-10 upper=10 effort=1000 velocity=0.5
- joint rail_z_default: limit lower=-2.5 upper=2.5 effort=1000 velocity=0.5 -> lower=-10 upper=10 effort=1000 velocity=0.5
